Commit message: Legg til valgfri sensorstøy, vind og treghet i motorene
For å teste regulatorer mer realistisk kan dette nå slås på, hver for seg:
- sensor_noise: støy og fast skjevhet på gyro og akselerometer, og støy på
  GPS-posisjonen (tallene i parameters.xacro)
- wind_speed, wind_direction, wind_gust: vind med VRX sin USVWind i open_water
- thrust_time_constant: førsteordens treghet i thruster_adapter

Modellen og open_water lages fra xacro ved oppstart med valgene. Valgene finnes
i sim.launch.py og compose. Testet i Gazebo: støyen gir realistisk spredning,
vinden driver båten riktig vei, og tidskonstanten stemmer med teorien.
Gazebo tolker GPS-støy som grader, så sensors.xacro regner om fra meter.

Co-Authored-By: Claude Opus 5.5 <noreply@anthropic.com>

File: src/asv_gazebo/models/asv/model.sdf.xacro (robot description, xacro)
@@ -11,4 +11,7 @@
 -->
 <sdf version="1.9" xmlns:xacro="http://www.ros.org/wiki/xacro">
+  <!-- Valg når modellen lages (asv.launch.py sender dem videre fra sim.launch.py). -->
+  <xacro:arg name="sensor_noise" default="false"/>
+  <xacro:property name="sensor_noise" value="$(arg sensor_noise)"/>
   <xacro:include filename="xacro/parameters.xacro"/>
   <xacro:include filename="xacro/thrusters.xacro"/>

File: src/asv_gazebo/models/asv/xacro/parameters.xacro (robot description, xacro)
@@ -72,3 +72,12 @@
   <xacro:property name="gps_rate" value="20"/>
   <xacro:property name="gps_height" value="0.15"/>
+  <!-- Sensorstøy, brukt når modellen lages med sensor_noise:=true (standardavvik, hvit støy, og en
+       fast skjevhet som trekkes én gang per kjøring). ANSLAG for en MEMS-IMU og en GPS med
+       korreksjoner. Gazebo har ingen støy på IMU-ens orientering, så heading er fortsatt eksakt. -->
+  <xacro:property name="gyro_noise" value="0.002"/>        <!-- rad/s -->
+  <xacro:property name="gyro_bias" value="0.0005"/>        <!-- rad/s -->
+  <xacro:property name="accel_noise" value="0.02"/>        <!-- m/s2 -->
+  <xacro:property name="accel_bias" value="0.01"/>         <!-- m/s2 -->
+  <xacro:property name="gps_horizontal_noise" value="0.02"/>  <!-- m -->
+  <xacro:property name="gps_vertical_noise" value="0.04"/>    <!-- m -->
 </sdf>

File: src/asv_gazebo/models/asv/xacro/sensors.xacro (robot description, xacro)
@@ -1,8 +1,21 @@
 <?xml version="1.0"?>
 <!--
-  Sensorene som makroer. De settes inn i base_link i model.sdf.xacro. Nye sensorer (lidar,
-  kamera) legges til her og trenger en bro i asv.launch.py og en linje i sensor_relay sin config.
+  Sensorene som makroer. De settes inn i base_link i model.sdf.xacro. Med sensor_noise:=true får
+  IMU og GPS støy (tallene i parameters.xacro). Nye sensorer (lidar, kamera) legges til her og
+  trenger en bro i asv.launch.py og en linje i sensor_relay sin config.
 -->
 <sdf xmlns:xacro="http://www.ros.org/wiki/xacro">
+  <!-- Gaussisk støy med fast skjevhet (bias) på én akse. -->
+  <xacro:macro name="noise" params="stddev bias">
+    <noise type="gaussian">
+      <mean>0</mean><stddev>${stddev}</stddev>
+      <bias_mean>0</bias_mean><bias_stddev>${bias}</bias_stddev>
+    </noise>
+  </xacro:macro>
+  <xacro:macro name="xyz_noise" params="stddev bias">
+    <x><xacro:noise stddev="${stddev}" bias="${bias}"/></x>
+    <y><xacro:noise stddev="${stddev}" bias="${bias}"/></y>
+    <z><xacro:noise stddev="${stddev}" bias="${bias}"/></z>
+  </xacro:macro>
   <xacro:macro name="imu">
     <sensor name="imu" type="imu">
@@ -14,4 +27,8 @@
           <localization>ENU</localization>
         </orientation_reference_frame>
+        <xacro:if value="${sensor_noise}">
+          <angular_velocity><xacro:xyz_noise stddev="${gyro_noise}" bias="${gyro_bias}"/></angular_velocity>
+          <linear_acceleration><xacro:xyz_noise stddev="${accel_noise}" bias="${accel_bias}"/></linear_acceleration>
+        </xacro:if>
       </imu>
     </sensor>
@@ -23,4 +40,13 @@
       <update_rate>${gps_rate}</update_rate>
       <topic>/asv/sensors/gps</topic>
+      <xacro:if value="${sensor_noise}">
+        <navsat>
+          <position_sensing>
+            <!-- Gazebo tolker horisontal støy som grader breddegrad/lengdegrad, ikke meter. -->
+            <horizontal><xacro:noise stddev="${gps_horizontal_noise / 111320.0}" bias="0"/></horizontal>
+            <vertical><xacro:noise stddev="${gps_vertical_noise}" bias="0"/></vertical>
+          </position_sensing>
+        </navsat>
+      </xacro:if>
     </sensor>
   </xacro:macro>

File: src/asv_gazebo/worlds/open_water.sdf.xacro (robot description, xacro)
@@ -7,4 +7,15 @@
 -->
 <sdf version="1.9" xmlns:xacro="http://www.ros.org/wiki/xacro">
+  <!-- Valg når verdenen lages (asv.launch.py sender dem videre fra sim.launch.py).
+       wind_speed: middelvind i m/s, 0 = ingen vind. wind_direction: retningen vinden blåser mot,
+       i grader (0 = mot øst, 90 = mot nord). wind_gust: hvor mye vinden varierer (0 = jevn). -->
+  <xacro:arg name="wind_speed" default="0"/>
+  <xacro:arg name="wind_direction" default="0"/>
+  <xacro:arg name="wind_gust" default="0"/>
+  <xacro:property name="wind_speed" value="$(arg wind_speed)"/>
+  <!-- Vindkraften på båten (VRX USVWind): F = koeffisient * relativ vindfart * |relativ vindfart|,
+       per akse i verden. ANSLAG: 0,5 * lufttetthet * Cd * areal over vannet (ca. 1,5 x 0,27 m
+       fra siden), Cd ca. 1. -->
+  <xacro:property name="wind_coeff" value="0.15 0.15 0.05"/>
   <!-- GPS-posisjonen til origo -->
   <xacro:property name="latitude" value="-33.722768768890596"/>
@@ -77,4 +88,21 @@
       </message>
     </plugin>
+    <xacro:if value="${float(wind_speed) > 0}">
+      <plugin filename="libUSVWind.so" name="vrx::USVWind">
+        <wind_obj>
+          <name>asv</name>
+          <link_name>base_link</link_name>
+          <coeff_vector>${wind_coeff}</coeff_vector>
+        </wind_obj>
+        <wind_direction>$(arg wind_direction)</wind_direction>
+        <wind_mean_velocity>${wind_speed}</wind_mean_velocity>
+        <var_wind_gain_constants>$(arg wind_gust)</var_wind_gain_constants>
+        <var_wind_time_constants>2</var_wind_time_constants>
+        <random_seed>10</random_seed>
+        <update_rate>10</update_rate>
+        <topic_wind_speed>/vrx/debug/wind/speed</topic_wind_speed>
+        <topic_wind_direction>/vrx/debug/wind/direction</topic_wind_direction>
+      </plugin>
+    </xacro:if>
   </world>
 </sdf>

Commit message: Rett bølgene: båten følger dem, og bildet stemmer med fysikken
- Oppdriften er delt i et rutenett av bokser (4 x 2). VRX regner vannet som
  flatt rundt hvert element, så med én boks gikk båten bare opp og ned. Nå
  ruller og stamper den med bølgene. Dypgangen i stille vann er uendret.
- Vannet i open_water har bølgeparametrene i <wavefield>, fordi VRX sin
  WaveVisual låser seg til standardbølgene før topicen kommer.
- Eget vannmesh (ocean.obj, scripts/make_ocean_mesh.py) med 1 m mellom
  punktene rundt båten. VRX sitt har 19 m, og da så båten ut som den gikk
  gjennom bølgene.
- wave_height (største utslag i meter) erstatter wave_gain, som ikke er en
  høyde. Omregnet med VRX sin formel i asv_gazebo/waves.py.

Co-Authored-By: Claude Opus 5.5 <noreply@anthropic.com>

File: src/asv_gazebo/models/asv/model.sdf.xacro (robot description, xacro)
@@ -67,4 +67,21 @@
     <xacro:steerable_thruster side="right" y_sign="-1"/>
     <xacro:bow_thruster/>
+    <!-- Oppdrift: rutenettet av bokser fra parameters.xacro, én <buoyancy> per boks. -->
+    <xacro:macro name="buoyancy_grid" params="cells">
+      <xacro:if value="${len(cells) > 0}">
+        <xacro:property name="i" value="${cells[0][0]}"/>
+        <xacro:property name="j" value="${cells[0][1]}"/>
+        <xacro:property name="dx" value="${buoyancy_length / buoyancy_nx}"/>
+        <xacro:property name="dy" value="${buoyancy_width / buoyancy_ny}"/>
+        <buoyancy name="hull_buoyancy_${i}_${j}">
+          <link_name>base_link</link_name>
+          <pose>${buoyancy_x - buoyancy_length / 2 + dx * (i + 0.5)} ${-buoyancy_width / 2 + dy * (j + 0.5)} ${buoyancy_z} 0 0 0</pose>
+          <geometry>
+            <box><size>${dx} ${dy} ${buoyancy_height}</size></box>
+          </geometry>
+        </buoyancy>
+        <xacro:buoyancy_grid cells="${cells[1:]}"/>
+      </xacro:if>
+    </xacro:macro>
     <plugin name="vrx::PolyhedraBuoyancyDrag" filename="libPolyhedraBuoyancyDrag.so">
       <fluid_density>1000</fluid_density>
@@ -74,11 +91,5 @@
       <linear_drag>0.0</linear_drag>
       <angular_drag>0.0</angular_drag>
-      <buoyancy name="hull_buoyancy">
-        <link_name>base_link</link_name>
-        <pose>${buoyancy_pose} 0 0 0</pose>
-        <geometry>
-          <box><size>${buoyancy_size}</size></box>
-        </geometry>
-      </buoyancy>
+      <xacro:buoyancy_grid cells="${[(i, j) for i in python.range(buoyancy_nx) for j in python.range(buoyancy_ny)]}"/>
       <wavefield>
         <topic>/vrx/wavefield/parameters</topic>

File: src/asv_gazebo/models/asv/xacro/parameters.xacro (robot description, xacro)
@@ -17,6 +17,15 @@
        som skroget. Bunnen er lagt slik at dypgangen stemmer for masser mellom 40 og 50 kg.
        Utenfor det spennet må boksen regnes ut på nytt. -->
-  <xacro:property name="buoyancy_pose" value="-0.19 0 -0.051"/>
-  <xacro:property name="buoyancy_size" value="1.12 0.52 0.342"/>
+  <xacro:property name="buoyancy_x" value="-0.19"/>
+  <xacro:property name="buoyancy_z" value="-0.051"/>
+  <xacro:property name="buoyancy_length" value="1.12"/>
+  <xacro:property name="buoyancy_width" value="0.52"/>
+  <xacro:property name="buoyancy_height" value="0.342"/>
+  <!-- Boksen deles i et rutenett (antall langs og på tvers). VRX regner vannet som flatt rundt hver
+       boks, med høyden i midten av boksen. Med én boks går båten bare opp og ned i bølgene. Med flere
+       kjenner den at vannet heller, og ruller og stamper. Samlet størrelse er den samme, så
+       dypgangen i stille vann endres ikke. -->
+  <xacro:property name="buoyancy_nx" value="4"/>
+  <xacro:property name="buoyancy_ny" value="2"/>
   <!-- Angrepspunktet for motstanden i vannet, 6 cm bak tyngdepunktet. ANSLAG: skrogets
        lateralplan har senter ved x = -0,05, men thrusterne og stagene akter virker som finner og

File: src/asv_gazebo/worlds/open_water.sdf.xacro (robot description, xacro)
@@ -21,10 +21,16 @@
   <xacro:property name="latitude" value="-33.722768768890596"/>
   <xacro:property name="longitude" value="150.67399110173986"/>
-  <!-- Bølger (Gerstner-bølger i VRX). gain er omtrent bølgehøyden i meter, period i sekunder,
-       direction i radianer, steepness 0-1. Samme som sydney_regatta. -->
-  <xacro:property name="wave_gain" value="0.3"/>
-  <xacro:property name="wave_period" value="5"/>
-  <xacro:property name="wave_direction" value="0.0"/>
-  <xacro:property name="wave_steepness" value="0"/>
+  <!-- Bølger (Gerstner-bølger i VRX), valg ved oppstart. wave_gain er en skaleringsfaktor i VRX sin
+       bølgemodell (Pierson-Moskowitz), ikke høyden. asv.launch.py regner den ut fra wave_height
+       (største utslag i meter). wave_period i sekunder, wave_direction i radianer, wave_steepness
+       0-1. Standard er som sydney_regatta (gain 0,3, periode 5 s, største utslag ca. 0,11 m). -->
+  <xacro:arg name="wave_gain" default="0.3"/>
+  <xacro:arg name="wave_period" default="5"/>
+  <xacro:arg name="wave_direction" default="0.0"/>
+  <xacro:arg name="wave_steepness" default="0"/>
+  <xacro:property name="wave_gain" value="$(arg wave_gain)"/>
+  <xacro:property name="wave_period" value="$(arg wave_period)"/>
+  <xacro:property name="wave_direction" value="$(arg wave_direction)"/>
+  <xacro:property name="wave_steepness" value="$(arg wave_steepness)"/>
   <xacro:macro name="wave_param" params="key value">
     params {
@@ -73,10 +79,44 @@
       <direction>-0.5 0.1 -0.9</direction>
     </light>
-    <!-- Vannflaten fra VRX, 6 x 6 km. -->
-    <include>
-      <name>water</name>
-      <pose>0 0 0 0 0 0</pose>
-      <uri>coast_waves</uri>
-    </include>
+    <!-- Vannflaten, 6 x 6 km: VRX sin coast_waves, men skrevet inn her med bølgeparametrene i
+         <wavefield>. WaveVisual sender bølgene til grafikkortet bare én gang, før parametrene på
+         topicen kommer. Uten dette viser bildet VRX sine standardbølger (gain 1, periode 5 s), mens
+         fysikken bruker de riktige, og båten ser ut som den er under vann. -->
+    <model name="water">
+      <static>true</static>
+      <link name="link">
+        <visual name="wave_visual">
+          <!-- Eget mesh med 1 m mellom punktene rundt båten (scripts/make_ocean_mesh.py). VRX sitt
+               har ca. 19 m, og da tegnes bølgene rundt en så liten båt helt feil. -->
+          <geometry><mesh><uri>model://ocean/meshes/ocean.obj</uri></mesh></geometry>
+          <plugin filename="libWaveVisual.so" name="vrx::WaveVisual">
+            <shader>
+              <vertex>model://coast_waves/materials/programs/GerstnerWaves_vs_330.glsl</vertex>
+              <fragment>model://coast_waves/materials/programs/GerstnerWaves_fs_330.glsl</fragment>
+              <parameters>
+                <rescale>0.125</rescale>
+                <bumpScale>75 75</bumpScale>
+                <bumpSpeed>0.01 0.0</bumpSpeed>
+                <hdrMultiplier>0.4</hdrMultiplier>
+                <fresnelPower>5.0</fresnelPower>
+                <shallowColor>0 0.1 0.2 1.0</shallowColor>
+                <deepColor>0 0.05 0.2 1.0</deepColor>
+              </parameters>
+            </shader>
+            <wavefield>
+              <topic>/vrx/wavefield/parameters</topic>
+              <wave>
+                <model>PMS</model>
+                <period>${wave_period}</period>
+                <direction>${wave_direction}</direction>
+                <steepness>${wave_steepness}</steepness>
+                <gain>${wave_gain}</gain>
+              </wave>
+            </wavefield>
+          </plugin>
+          <visibility_flags>8</visibility_flags>
+        </visual>
+      </link>
+    </model>
     <!-- Bølgene. Oppdriften til båten og bøyene leser dem fra samme topic. -->
     <plugin filename="libPublisherPlugin.so" name="vrx::PublisherPlugin">

Commit message: Legg komponentene om bord i components.yaml, innenfor fast totalvekt
Totalvekten er nå fast (total_mass = 45 kg) med skrog, thrustere og alle
komponentene. Komponentene (batteri, elektronikk osv.) legges inn med masse,
plassering og størrelse i components.yaml, og skroget får massen som er
igjen. Da er dypgangen den samme, mens tyngdepunktet flytter seg etter hvor
komponentene står. For tunge komponenter stopper bygget med en feilmelding.

Før veide modellen 46,4 kg, fordi thrusterne kom i tillegg til skroget.
Testet i Gazebo: 45,00 kg uten komponenter, og et batteri på 8 kg langt bak
gir 3,7° akterlig trim.

Co-Authored-By: Claude Opus 5.5 <noreply@anthropic.com>

File: src/asv_gazebo/models/asv/model.sdf.xacro (robot description, xacro)
@@ -6,4 +6,6 @@
   - xacro/thrusters.xacro: thrusterne
   - xacro/sensors.xacro: sensorene
+  - components.yaml: komponentene om bord (batteri, elektronikk osv.), innenfor totalvekten
+  - xacro/components.xacro: lager komponentene fra components.yaml
   Skrogfilen skrog10-1.stl er delt i skrog, thrusterhus og propeller (meshes/), slik at
   thrusterne dreier og propellene snurrer synlig. Meshene brukes bare til visning. Fysikken er
@@ -20,4 +22,14 @@
   <xacro:include filename="xacro/thrusters.xacro"/>
   <xacro:include filename="xacro/sensors.xacro"/>
+  <xacro:include filename="xacro/components.xacro"/>
+  <!-- Skroget får det som er igjen av totalvekten, så totalen alltid er total_mass. -->
+  <xacro:property name="fixed_parts_mass" value="${2 * pod_mass + 3 * prop_mass + hydro_mass}"/>
+  <xacro:property name="hull_mass" value="${total_mass - components_mass - fixed_parts_mass}"/>
+  <xacro:if value="${hull_mass &lt;= 0}">
+    ${xacro.error('Komponentene i components.yaml (%.1f kg) og thrusterne (%.1f kg) veier mer enn total_mass (%.1f kg).' % (components_mass, fixed_parts_mass, total_mass))}
+    <!-- xacro.error stopper ikke, så navnet under (som ikke finnes) stopper xacro og bygget. -->
+    ${STOPP_komponentene_er_for_tunge}
+  </xacro:if>
+  <xacro:property name="hull_share" value="${hull_mass / total_mass}"/>
   <model name="asv">
     <link name="base_link">
@@ -26,5 +38,5 @@
         <mass>${hull_mass}</mass>
         <inertia>
-          <ixx>${hull_ixx}</ixx><iyy>${hull_iyy}</iyy><izz>${hull_izz}</izz>
+          <ixx>${hull_ixx * hull_share}</ixx><iyy>${hull_iyy * hull_share}</iyy><izz>${hull_izz * hull_share}</izz>
           <ixy>0</ixy><ixz>0</ixz><iyz>0</iyz>
         </inertia>
@@ -56,5 +68,5 @@
       <pose>${hydro_pose} 0 0 0</pose>
       <inertial>
-        <mass>0.1</mass>
+        <mass>${hydro_mass}</mass>
         <inertia><ixx>0.0001</ixx><iyy>0.0001</iyy><izz>0.0001</izz><ixy>0</ixy><ixz>0</ixz><iyz>0</iyz></inertia>
       </inertial>
@@ -64,4 +76,6 @@
       <child>hydro_link</child>
     </joint>
+    <!-- Komponentene fra components.yaml (batteri, elektronikk osv.). -->
+    <xacro:all_components items="${components}"/>
     <xacro:steerable_thruster side="left" y_sign="1"/>
     <xacro:steerable_thruster side="right" y_sign="-1"/>

File: src/asv_gazebo/models/asv/xacro/parameters.xacro (robot description, xacro)
@@ -6,9 +6,12 @@
 -->
 <sdf xmlns:xacro="http://www.ros.org/wiki/xacro">
-  <!-- Skroget. ANSLAG: 45 kg, midt i spennet 40-50 kg. Gir vannlinje ved z = -0,145
-       (dypgang 10,5 cm). 40 kg gir z = -0,153 og 50 kg gir z = -0,136. -->
-  <xacro:property name="hull_mass" value="45.0"/>
+  <!-- Totalvekten med alt (skrog, thrustere og komponentene i components.yaml), anslått til 45 kg.
+       Gir vannlinje ved z = -0,145 (dypgang 10,5 cm). 40 kg gir z = -0,153 og 50 kg gir z = -0,136.
+       Skroget får massen som er igjen etter thrusterne og komponentene (model.sdf.xacro). -->
+  <xacro:property name="total_mass" value="45.0"/>
+  <!-- Tyngdepunktet til skroget og alt som ikke er lagt inn som egen komponent. ANSLAG. -->
   <xacro:property name="hull_cog" value="-0.19 0 -0.12"/>
-  <!-- Treghetsmomentet er regnet som en massiv boks. -->
+  <!-- Treghetsmomentet for hele båten (45 kg), regnet som en massiv boks. Skroget får en andel
+       etter massen sin, og komponentene legger til sitt eget der de står. -->
   <xacro:property name="hull_ixx" value="1.24"/>
   <xacro:property name="hull_iyy" value="7.65"/>
@@ -67,4 +70,9 @@
   <xacro:property name="stern_min_thrust" value="-30"/>
   <xacro:property name="stern_prop_diameter" value="0.09"/>
+  <!-- Massen til thrusterhusene og propellene (egne deler i modellen, regnet med i total_mass). -->
+  <xacro:property name="pod_mass" value="0.5"/>
+  <xacro:property name="prop_mass" value="0.1"/>
+  <!-- Punktet vannmotstanden angriper i er en egen del med litt masse (Gazebo krever det). -->
+  <xacro:property name="hydro_mass" value="0.1"/>
   <!-- Dreiing: +-90° er bekreftet (control, 2026-10-19), og grensen ligger i thruster_adapter.
        Leddet tillater litt mer, for et ledd som kjøres helt i stopp, låser seg.

File: src/asv_gazebo/models/asv/xacro/thrusters.xacro (robot description, xacro)
@@ -55,10 +55,10 @@
       <pose>${pose}</pose>
       <xacro:dark_visual name="${side}_pod_visual" mesh="${side}_pod.stl"/>
-      <xacro:small_inertial mass="0.5" inertia="0.001"/>
+      <xacro:small_inertial mass="${pod_mass}" inertia="0.001"/>
     </link>
     <link name="${side}_prop_link">
       <pose>${pose}</pose>
       <xacro:dark_visual name="${side}_rotor_visual" mesh="${side}_rotor.stl"/>
-      <xacro:small_inertial mass="0.1" inertia="0.0001"/>
+      <xacro:small_inertial mass="${prop_mass}" inertia="0.0001"/>
     </link>
     <joint name="${side}_pod_joint" type="revolute">
@@ -88,5 +88,5 @@
     <link name="bow_prop_link">
       <pose>${bow_x} 0 ${bow_z} 0 0 0</pose>
-      <xacro:small_inertial mass="0.1" inertia="0.0001"/>
+      <xacro:small_inertial mass="${prop_mass}" inertia="0.0001"/>
     </link>
     <joint name="bow_prop_joint" type="revolute">
