Commit message: Legg til lidar og kamera med plassering i components.yaml
Sensorer legges i components.yaml under sensors:, med type (lidar eller
camera), plassering, vinkel og vekt, som regnes inn i totalvekten på 45 kg.
Gazebo-sensorene lages av xacro, og asv.launch.py lager broene til
/autonomy/lidar/<navn>/... og /autonomy/camera/<navn>/... fra den samme fila.
Valgfrie felt (rekkevidde, oppløsning, synsfelt) har standardverdier.

Testet med en lidar og et kamera: 10 Hz og 15 Hz, kameraet ser slalåmbøyene,
og simulatoren går på 0,99 av sanntid. Lista er tom som standard.

Co-Authored-By: Claude Opus 5.5 <noreply@anthropic.com>

File: src/asv_gazebo/models/asv/model.sdf.xacro (robot description, xacro)
@@ -27,5 +27,5 @@
   <xacro:property name="hull_mass" value="${total_mass - components_mass - fixed_parts_mass}"/>
   <xacro:if value="${hull_mass &lt;= 0}">
-    ${xacro.error('Komponentene i components.yaml (%.1f kg) og thrusterne (%.1f kg) veier mer enn total_mass (%.1f kg).' % (components_mass, fixed_parts_mass, total_mass))}
+    ${xacro.error('Komponentene og sensorene i components.yaml (%.1f kg) og thrusterne (%.1f kg) veier mer enn total_mass (%.1f kg).' % (components_mass, fixed_parts_mass, total_mass))}
     <!-- xacro.error stopper ikke, så navnet under (som ikke finnes) stopper xacro og bygget. -->
     ${STOPP_komponentene_er_for_tunge}
@@ -78,4 +78,6 @@
     <!-- Komponentene fra components.yaml (batteri, elektronikk osv.). -->
     <xacro:all_components items="${components}"/>
+    <!-- Sensorene fra components.yaml (lidar, kamera), med plassering. -->
+    <xacro:all_sensors items="${sensors}"/>
     <xacro:steerable_thruster side="left" y_sign="1"/>
     <xacro:steerable_thruster side="right" y_sign="-1"/>

File: src/asv_gazebo/models/asv/xacro/components.xacro (robot description, xacro)
@@ -1,11 +1,17 @@
 <?xml version="1.0"?>
 <!--
-  Komponentene fra components.yaml (stien regnes fra model.sdf.xacro): én del per komponent, festet til skroget, med masse,
-  treghetsmoment (massiv boks) og en enkel boks som vises i Gazebo. Ingen kollisjon, de er inne i skroget.
+  Komponentene og sensorene fra components.yaml (stien regnes fra model.sdf.xacro). Hver blir en
+  del festet til skroget, med masse, treghetsmoment (massiv boks) og en enkel boks som vises i
+  Gazebo. Ingen kollisjon, de er inne i eller oppå skroget. Sensorene får i tillegg en Gazebo-sensor.
+  asv.launch.py leser den samme fila og lager broene til ROS for sensorene.
 -->
 <sdf xmlns:xacro="http://www.ros.org/wiki/xacro">
-  <xacro:property name="components" value="${xacro.load_yaml('components.yaml')['components'] or []}"/>
-  <xacro:property name="components_mass" value="${math.fsum([c['mass'] for c in components])}"/>
-  <xacro:macro name="component" params="name mass x y z size">
+  <xacro:property name="config" value="${xacro.load_yaml('components.yaml')}"/>
+  <xacro:property name="components" value="${config.get('components') or []}"/>
+  <xacro:property name="sensors" value="${config.get('sensors') or []}"/>
+  <xacro:property name="components_mass"
+                  value="${math.fsum([c['mass'] for c in components] + [s['mass'] for s in sensors])}"/>
+  <!-- Del med masse og en boks som vises. Innholdet i makroen (f.eks. en sensor) legges i delen. -->
+  <xacro:macro name="part" params="name mass x y z size color **content">
     <xacro:property name="l" value="${size[0]}"/>
     <xacro:property name="b" value="${size[1]}"/>
@@ -25,8 +31,9 @@
         <geometry><box><size>${l} ${b} ${h}</size></box></geometry>
         <material>
-          <ambient>0.9 0.5 0.1 1</ambient>
-          <diffuse>0.9 0.5 0.1 1</diffuse>
+          <ambient>${color}</ambient>
+          <diffuse>${color}</diffuse>
         </material>
       </visual>
+      <xacro:insert_block name="content"/>
     </link>
     <joint name="${name}_joint" type="fixed">
@@ -39,8 +46,74 @@
     <xacro:if value="${len(items) > 0}">
       <xacro:property name="c" value="${items[0]}"/>
-      <xacro:component name="${c['name']}" mass="${c['mass']}" x="${c['x']}" y="${c['y']}"
-                       z="${c['z']}" size="${c['size']}"/>
+      <xacro:part name="${c['name']}" mass="${c['mass']}" x="${c['x']}" y="${c['y']}" z="${c['z']}"
+                  size="${c['size']}" color="0.9 0.5 0.1 1">
+        <content/>
+      </xacro:part>
       <xacro:all_components items="${items[1:]}"/>
     </xacro:if>
   </xacro:macro>
+  <!--
+    Sensorer. Vinklene (roll, pitch, yaw) er i grader. Kameraet ser langs x i sin egen ramme, og
+    lidaren skanner rundt z. Standardverdiene under brukes når feltet mangler i components.yaml.
+    Gazebo-topics: /asv/sensors/<navn>/scan (lidar) og /asv/sensors/<navn>/image_raw (kamera).
+  -->
+  <xacro:macro name="all_sensors" params="items">
+    <xacro:if value="${len(items) > 0}">
+      <xacro:property name="s" value="${items[0]}"/>
+      <xacro:property name="deg" value="${math.pi / 180.0}"/>
+      <xacro:unless value="${s['type'] in ('lidar', 'camera')}">
+        ${xacro.error('Sensoren %s i components.yaml har type %s. Kjente typer: lidar, camera.' % (s['name'], s['type']))}
+        ${STOPP_ukjent_sensortype}
+      </xacro:unless>
+      <xacro:part name="${s['name']}" mass="${s['mass']}" x="${s['x']}" y="${s['y']}" z="${s['z']}"
+                  size="${s.get('size', [0.08, 0.08, 0.08])}" color="0.1 0.1 0.1 1">
+        <content>
+          <sensor name="${s['name']}" type="${'gpu_lidar' if s['type'] == 'lidar' else 'camera'}">
+            <pose>0 0 0 ${s.get('roll', 0) * deg} ${s.get('pitch', 0) * deg} ${s.get('yaw', 0) * deg}</pose>
+            <always_on>1</always_on>
+            <xacro:if value="${s['type'] == 'lidar'}">
+              <update_rate>${s.get('rate', 10)}</update_rate>
+              <topic>/asv/sensors/${s['name']}/scan</topic>
+              <lidar>
+                <scan>
+                  <horizontal>
+                    <samples>${s.get('samples', 360)}</samples>
+                    <min_angle>${-s.get('fov_horizontal', 360) / 2.0 * deg}</min_angle>
+                    <max_angle>${s.get('fov_horizontal', 360) / 2.0 * deg}</max_angle>
+                  </horizontal>
+                  <vertical>
+                    <samples>${s.get('vertical_samples', 16)}</samples>
+                    <min_angle>${-s.get('fov_vertical', 30) / 2.0 * deg}</min_angle>
+                    <max_angle>${s.get('fov_vertical', 30) / 2.0 * deg}</max_angle>
+                  </vertical>
+                </scan>
+                <range>
+                  <min>${s.get('range_min', 0.3)}</min>
+                  <max>${s.get('range_max', 50.0)}</max>
+                  <resolution>0.01</resolution>
+                </range>
+              </lidar>
+            </xacro:if>
+            <xacro:if value="${s['type'] == 'camera'}">
+              <update_rate>${s.get('rate', 15)}</update_rate>
+              <topic>/asv/sensors/${s['name']}/image_raw</topic>
+              <camera>
+                <horizontal_fov>${s.get('fov_horizontal', 80) * deg}</horizontal_fov>
+                <image>
+                  <width>${s.get('width', 640)}</width>
+                  <height>${s.get('height', 480)}</height>
+                  <format>R8G8B8</format>
+                </image>
+                <clip>
+                  <near>${s.get('near', 0.1)}</near>
+                  <far>${s.get('far', 100.0)}</far>
+                </clip>
+              </camera>
+            </xacro:if>
+          </sensor>
+        </content>
+      </xacro:part>
+      <xacro:all_sensors items="${items[1:]}"/>
+    </xacro:if>
+  </xacro:macro>
 </sdf>
